File: Meter hardware design/PCB CAD Design/EnAcess PCB.kicad_pcb (KiCad board)
At the start: 2 copper layers, 162.6 x 147.3 mm, 156 parts, among them J1 RTC, J10 curr, J11 , J12 RS232, J13 6v BAT, J14 Conn_01x01, J15 Conn_01x01, J16 Conn_01x01, J2 LCD pinout, J3 4x4 keypad, J4 Cicada GSM module, J5 , J6 , J7 relay, J8 220VAC.in, J9 LED_socket, Q1 BC547, Q2 BC547, Q3 IRF460, Q4 BC547, Q5 BC547, Q6 BC547, U1 UC3843_DIP8, U2 L7805, U3 PC817, U4 PC817, U5 LM350, U6 TL431LP, U7 LM350, U8 ATM90E26, U9 PC817

Commit message: PCB review (#8)
* Delete EnAcess PCB.kicad_sch-bak

* Delete Meter hardware design/PCB CAD Design directory

* Create CAD

* Add files via upload

* Delete Meter hardware design/production file directory

* Create pro

* Add files via upload
Parts:
- removed Q1, Q4, Q5, Q6: BC547, Package_TO_SOT_THT:TO-92_Inline_Wide
- removed R52: 470R, Resistor_THT:R_Axial_DIN0207_L6.3mm_D2.5mm_P10.16mm_Horizontal
- removed R53, R56, R57: 1K, Resistor_THT:R_Axial_DIN0207_L6.3mm_D2.5mm_P10.16mm_Horizontal
- removed U3, U9: PC817, Package_DIP:DIP-4_W7.62mm
- added C44: 104, Capacitor_THT:C_Disc_D10.0mm_W2.5mm_P5.00mm, F.Cu at (45.8, 141.4)
- added D10: 1n5819, Diode_THT:D_DO-34_SOD68_P7.62mm_Horizontal, F.Cu at (42.4, 47.0)
- added D13: 1n5819, Diode_THT:D_DO-34_SOD68_P7.62mm_Horizontal, F.Cu at (96.0, 27.0)
- added D20: D_Zener, Diode_THT:D_A-405_P12.70mm_Horizontal, F.Cu at (62.2, 27.5)
- added D9: D_Zener, Diode_THT:D_A-405_P12.70mm_Horizontal, F.Cu at (25.9, 46.8)
- added J17: 6v BAT, Connector_JST:JST_EH_S2B-EH_1x02_P2.50mm_Horizontal, F.Cu at (58.1, 52.5)
- added U10: L293, Package_DIP:DIP-16_W7.62mm, F.Cu at (50.6, 130.1)
- D6: value 1n4007 -> 1n4148
- D8: value 12v/1W Zener -> 12vZ
- R11: value 1K -> 470R
- R4: value 470R -> 10R
- moved R11 101.9 mm to (75.1, 41.6), turned to 180 degrees
- moved R4 75.6 mm to (56.8, 31.9), turned to -90 degrees
- moved R3 1.57 mm to (42.1, 18.0)
- moved J13 1.34 mm to (67.3, 22.3)
- moved D1 1.16 mm to (58.5, 18.0)
- moved R39 0.61 mm to (74.5, 16.6)
- moved C4 0.53 mm to (96.2, 32.2)
Connections:
- D2 pad 2: +5V -> Net-(D13-A)
- R11 pad 1: con A -> +12V
- R11 pad 2: Net-(Q1-B) -> Net-(D10-A)
- R4 pad 1: REL_a -> +5V
- R4 pad 2: Net-(R4-Pad2) -> Net-(D10-A)
- U2 pad 3: +5V -> Net-(D13-A)
Routing:
- net con A: track 131.7 -> 0.00 mm
- net Net-(R52-Pad2): track 112.3 -> 0.00 mm, vias 2 -> 0
- net REL_b: track 5.41 -> 113.5 mm, vias 0 -> 2
- net con B: track 76.8 -> 0.00 mm, vias 1 -> 0
- net 12V_S: track 196.5 -> 262.4 mm
- net +12V: track 245.5 -> 199.2 mm
- net Net-(J7-Pin_2): track 36.6 -> 73.1 mm
- net Net-(D10-A): track 0.00 -> 26.7 mm
- net +5V: track 399.8 -> 379.8 mm
- net REL_a: track 69.9 -> 89.0 mm, vias 0 -> 1
- net Net-(R4-Pad2): track 16.5 -> 0.00 mm
- net Net-(D13-A): track 0.00 -> 16.4 mm
- net Net-(J7-Pin_1): track 55.3 -> 65.0 mm, vias 2 -> 0
- net Net-(Q1-B): track 4.76 -> 0.00 mm
- net Net-(Q6-B): track 4.68 -> 0.00 mm
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Other:
- board text removed: "470uf/10v"
